Commit message: - Updated main to set start/end time by frame number rather than time  - Updated Dagu5 model to prevent track sliding off  - Raygrid now dumps diff images  - Tweaked track scaling in TrackedVehicle

File: data/urdf/Dagu5.urdf (robot description, URDF)
Before this commit: robot Dagu5, 9 links, 8 joints
Links:
- added link link_Cube; collision box size=5.026439 0.104412 0.760734
- added link link_Cube.001; collision box size=5.026439 0.104412 0.760734
- link link_bl_Leg: geometry collision box size=1.837332 0.298121 0.712926; visual mesh filename=meshes/Cube.003.obj scale=0.68 0.126 0.353675
- link link_br_Leg: geometry collision box size=1.837332 0.297859 0.712926; visual mesh filename=meshes/Cube.006.obj scale=0.68 0.126 0.353675
- link link_fr_Leg: geometry collision box size=1.837831 0.297859 0.712926; visual mesh filename=meshes/Cube.005.obj scale=0.680185 0.126 0.353675
Joints:
- added joint link_Cube: type fixed, parent link_Body, child link_Cube, origin xyz=0.015789 1.920648 -0.852022 rpy=-3.141593 0 0
- added joint link_Cube.001: type fixed, parent link_Body, child link_Cube.001, origin xyz=0.015789 -2.0 -0.852022 rpy=-3.141593 0 0

Commit message: commit after OS crash - minor tweaks to vehcile tracks and terrain

File: data/urdf/Dagu5.urdf (robot description, URDF)
Before this commit: robot Dagu5, 11 links, 10 joints
Links:
- link link_Cube: geometry collision box size=5.526439 0.104412 1.760734
- link link_Cube.001: geometry collision box size=5.526439 0.104412 1.760734
- link link_br_Leg: geometry collision box size=1.837332 0.389566 0.712926; visual mesh filename=meshes/Cube.006.obj scale=0.68 0.126 0.353675
- link link_fr_Leg: geometry collision box size=1.837831 0.379697 0.712926; visual mesh filename=meshes/Cube.005.obj scale=0.680185 0.126 0.353675

Commit message: Switched from particle terrain to chrono::vehicle terrain Disabled raygrid Disabled particlesystem Added map XY scaling Refactored some code

File: data/urdf/Dagu5.urdf (robot description, URDF)
Before this commit: robot Dagu5, 11 links, 10 joints
Links:
- link link_Body: mass 500.0 -> 5000.0
- link link_bl_Leg: mass 20.0 -> 200.0
- link link_bl_Wheel: mass 10.0 -> 100.0
- link link_br_Leg: mass 20.0 -> 200.0
- link link_br_Wheel: mass 10.0 -> 100.0
- link link_fl_Leg: mass 20.0 -> 200.0
- link link_fl_Wheel: mass 10.0 -> 100.0
- link link_fr_Leg: mass 20.0 -> 200.0
- link link_fr_Wheel: mass 10.0 -> 100.0
